File: templates/jlcpcb-6layer/jlcpcb-6layer.kicad_pcb (KiCad board)
At the start: 6 copper layers, 0 parts

Commit message: [jlc] update with current 6 layer stackup info
Other:
- board outline added: 100 x 100 mm
Changed lines of the file:
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@@
 	(generator_version "10.0")
 	(general
-		(thickness 1.6)
+		(thickness 1.549)
 		(legacy_teardrops no)
 	)
@@
 				(type "prepreg")
 				(thickness 0.0994)
-				(material "FR4")
-				(epsilon_r 4.5)
+				(material "FR4 3313")
+				(epsilon_r 4.1)
 				(loss_tangent 0.02)
 			)
@@
 				(type "core")
 				(thickness 0.55)
-				(material "FR4")
-				(epsilon_r 4.5)
+				(material "FR4 core")
+				(epsilon_r 4.6)
 				(loss_tangent 0.02)
 			)
@@
 			(layer "dielectric 3"
 				(type "prepreg")
-				(thickness 0.0994)
-				(material "FR4")
-				(epsilon_r 4.5)
+				(thickness 0.1088)
+				(material "FR4 2116")
+				(epsilon_r 4.16)
 				(loss_tangent 0.02)
 			)
@@
 				(type "core")
 				(thickness 0.55)
-				(material "FR4")
-				(epsilon_r 4.5)
+				(material "FR4 core")
+				(epsilon_r 4.6)
 				(loss_tangent 0.02)
 			)
@@
 				(type "prepreg")
 				(thickness 0.0994)
-				(material "FR4")
-				(epsilon_r 4.5)
+				(material "FR4 3313")
+				(epsilon_r 4.1)
 				(loss_tangent 0.02)
 			)
@@
 		)
 	)
+	(gr_rect
+		(start 40 40)
+		(end 140 140)
+		(stroke
+			(width 0.05)
+			(type solid)
+		)
+		(fill no)
+		(layer "Edge.Cuts")
+	)
 	(embedded_fonts no)
